File: block-diagram/block-diagram.kicad_sch (KiCad schematic)
At the start: 11 parts, among them SW1 SW_Push, SW2 SW_Push

Commit message: draft rev 0 work in progress
Parts:
- removed D1, D3: RGB, symbol Device:LED
- removed D2: ~, symbol Device:LED
- removed JP1: SolderJumper_2_Bridged, symbol Jumper:SolderJumper_2_Bridged
- added C1, C10, C11, C2, C3, C4, C5, C6, C7, C8, C9: 2.2u, symbol Device:C_Small
- added D1, D10, D13, D16, D17, D18, D19, D2, D22, D23, D24, D25, D26, D29, D3, D31, D32, D35, D36, D39, D42, D43, D44, D49, D50, D51, D6, D60, D61, D62, D7, D8: D_Schottky_Small, symbol Device:D_Schottky_Small
- added D11, D14, D20, D27, D33, D37, D40, D45, D54, D58, D65: Green, symbol Device:LED
- added D12, D15, D21, D28, D30, D34, D38, D4, D41, D46, D47, D48, D5, D52, D53, D55, D56, D57, D59, D63, D64, D66, D9: RGB, symbol Device:LED
- added Green2, Green3, Green5, Green6, Green7, Green8: ~, symbol Device:LED
- added JP1, JP12, JP17, JP19, JP2, JP20, JP23, JP26, JP29, JP3, JP32, JP33, JP34, JP35, JP4: SolderJumper_3_Bridged12, symbol Jumper:SolderJumper_3_Bridged12
- added JP10, JP11, JP13, JP14, JP15, JP16, JP18, JP21, JP22, JP24, JP25, JP27, JP28, JP30, JP31, JP36, JP37, JP5, JP6, JP7, JP8, JP9: SolderJumper_2_Bridged, symbol Jumper:SolderJumper_2_Bridged
- added Q1, Q2, Q3, Q4, Q5, Q7, Q8: NMOS, symbol Simulation_SPICE:NMOS
- added Q6, Q9: PMOS, symbol Simulation_SPICE:PMOS
- added R10, R104, R106, R116, R119, R130, R133, R17, R18, R20, R35, R37, R38, R45, R51, R52, R54, R57, R58, R59, R6, R60, R61, R67, R70, R71, R74, R75, R77, R8, R80, R86, R95, R97: 10K, symbol Device:R_Small
- added R100, R11, R127, R140, R141, R27, R32, R40, R49, R72, R87: 200, symbol Device:R_Small
- added R101, R113, R12, R126, R33, R41, R50, R73, R88: 1, symbol Device:R_Small
- added R102, R103, R105, R114, R115, R117, R128, R129, R13, R131, R14, R15, R29, R30, R34, R42, R43, R44, R47, R56, R64, R65, R68, R7, R79, R81, R82, R84, R85, R89, R90, R91: R_Small, symbol Device:R_Small
- added R107, R108, R109, R111, R120, R121, R122, R124, R134, R135, R136, R138, R139, R16, R19, R21, R22, R23, R25, R28, R31, R36, R39, R46, R48, R53, R55, R62, R63, R69, R76, R78, R83, R92, R93, R96, R98: 2.2K, symbol Device:R_Small
- added R110, R112, R123, R137, R24, R9: 100, symbol Device:R_Small
- added R118, R132: 100K?, symbol Device:R_Small
- added R125, R26, R94: M, symbol Device:R_Small
- added R66: 27, symbol Device:R_Small
- added R99: 220, symbol Device:R_Small
- added SW10, SW11, SW12, SW13, SW14, SW15, SW16, SW17, SW18, SW19, SW20, SW21, SW22, SW23, SW24, SW25, SW3, SW4, SW5, SW6, SW7, SW8, SW9: SW_Push, symbol Switch:SW_Push
- added U1, U2, U3, U4, U5, U6, U7, U8: LM285S-1.2, Package_SO:SOIC-8_3.9x4.9mm_P1.27mm, symbol Reference_Voltage:LM285S-1.2
- added U10, U9: 3V, Package_SO:SOIC-8_3.9x4.9mm_P1.27mm, symbol Reference_Voltage:LM285S-1.2
- added Y1, Y2, Y3, Y4, Y5, Y6, Y7, Y8: Crystal, symbol Device:Crystal
- R1: value R_Small -> M
- R2: value R_Small -> 200
- R3: value R_Small -> 1
Connections:
- net +3V3: now also D12.2 (A), D13.2 (A), D24.1 (K), D26.2 (A), D28.1 (K), D31.1 (K), D34.2 (A), D7.1 (K), D9.2 (A), JP10.2 (B), JP15.2 (B), JP21.2 (B), Q6.1 (D), Q6.3 (S), R18.1, R19.2, R20.1, R28.1, R29.1, R30.1, R31.1, R34.1, R51.1, R52.1, R53.2, R54.1, R55.1, R56.1, R57.1, R58.2, R60.1, R61.1, R62.2, R63.1, R64.1, R65.1, R67.1, R68.1, R69.2, R70.1; no longer R1.1, R2.1, R3.1, R4.1, R5.1
- net GND: now also C1.2, C10.2, C11.2, C2.2, C3.2, C4.2, C5.2, C6.2, C7.2, C8.2, C9.2, D10.2 (A), D17.2 (A), D2.2 (A), D23.2 (A), D25.2 (A), D32.2 (A), D35.2 (A), D43.2 (A), D50.2 (A), D61.2 (A), D8.2 (A), Green2.1 (K), Green3.1 (K), Green5.1 (K), Green6.1 (K), Green7.1 (K), Green8.1 (K), Q1.3 (S), Q2.3 (S), Q3.3 (S), Q4.3 (S), Q5.3 (S), Q7.3 (S), Q8.3 (S), SW11.1, SW13.1, SW16.1, SW18.1, SW21.1, SW23.1, SW25.1, SW4.1, SW6.1, SW8.1, U1.4 (A), U10.4 (A), U2.4 (A), U3.4 (A), U4.4 (A), U5.4 (A), U6.4 (A), U7.4 (A), U8.4 (A), U9.4 (A)
- net at R3.2: now also D3.1 (K)
- net at SW2.2: now also JP2.2 (C); no longer R2.2
- new net: D31.2 (A), D32.1 (K)
- new net: D30.2 (A), R58.1
- new net: D22.2 (A), D23.1 (K)
- new net: D11.2 (A), R19.1
- new net: D1.2 (A), D2.1 (K)
- new net: C2.1, R11.1, R12.1, U2.6 (K), U2.8 (K)
- new net: JP2.1 (A), R24.1
- new net: D56.2 (A), R116.2
- new net: C8.1, R100.1, R101.1, U7.6 (K), U7.8 (K)
- new net: D48.1 (K), Q1.1 (D)
- new net: D48.2 (A), R98.1
- new net: D52.2 (A), R104.2
- new net: Q4.1 (D), R57.2
- new net: Green7.2 (A), Q4.2 (G), Q5.2 (G), R51.2, R52.2, R55.2
- new net: JP37.1 (A), R138.1
- new net: D65.2 (A), R135.2
- new net: D20.2 (A), R16.1
- new net: C7.1, R87.1, R88.1, U6.6 (K), U6.8 (K)
- new net: C1.1, R32.1, R33.1, U1.6 (K), U1.8 (K)
- new net: D14.1 (K), R23.1, R24.2
- new net: Q2.2 (G), R112.2
- new net: Q3.2 (G), R9.2
- new net: JP8.1 (A), R25.1
- new net: D63.2 (A), R130.2
- new net: D40.2 (A), R46.1
- new net: C9.1, R2.1, R3.1, U8.6 (K), U8.8 (K)
- new net: D47.2 (A), R97.2
- new net: D19.1 (K), R12.2
- new net: Green2.2 (A), R36.2
- new net: D33.2 (A), R62.1
- new net: D64.1 (K), Q8.1 (D)
- new net: Q8.2 (G), R133.2
- new net: D10.1 (K), D6.2 (A)
- new net: C3.1, R49.1, R50.1, U3.6 (K), U3.8 (K)
- new net: D16.2 (A), D17.1 (K)
- new net: C5.1, R40.1, R41.1, U4.6 (K), U4.8 (K)
- new net: Green6.2 (A), R48.2
- new net: D42.2 (A), D43.1 (K)
- new net: D13.1 (K), R33.2
- new net: R61.2, SW18.2
- new net: JP28.1 (A), R96.1
- new net: D44.1 (K), R88.2
- new net: Green8.2 (A), R78.2
- new net: D37.2 (A), R76.1
- new net: C11.1, R126.1, R141.2, U10.6 (K), U10.8 (K)
- new net: D5.2 (A), R21.1
- new net: JP25.1 (A), R83.1
- new net: Green3.2 (A), R63.2
- new net: D39.1 (K), R41.2
- new net: JP31.1 (A), R111.1
- new net: JP35.1 (A), R137.1
- new net: JP35.2 (C), SW25.2
- new net: D49.2 (A), D50.1 (K)
- new net: JP6.1 (A), R39.1
- new net: D26.1 (K), R50.2
- new net: D51.1 (K), R101.2
- new net: D65.1 (K), R136.1, R137.2
- new net: JP16.1 (A), R31.2
- new net: C10.1, R113.1, R27.1, U9.6 (K), U9.8 (K)
- new net: JP32.1 (A), R110.1
- new net: D54.1 (K), R109.1, R110.2
- new net: R77.2, SW16.2
- new net: R47.2, R85.2, SW11.2
- new net: D53.1 (K), Q2.1 (D)
- new net: R99.1, SW21.2
- new net: D45.2 (A), R93.2
- new net: JP1.1 (A), R123.1
- new net: D58.1 (K), R122.1, R123.2
- new net: D14.2 (A), R22.2
- new net: D4.2 (A), R6.2
- new net: D62.1 (K), R126.2
- new net: Q9.1 (D), R127.1
- new net: JP9.1 (A), R34.2
- new net: JP22.1 (A), R69.1
- new net: D45.1 (K), R92.1, R99.2
- new net: R20.2, SW8.2
- new net: R54.2, SW13.2
- new net: D64.2 (A), R134.1
- new net: Green5.2 (A), R28.2
- new net: D57.1 (K), Q7.1 (D)
- new net: D57.2 (A), R120.1
- new net: D53.2 (A), R107.1
- new net: D36.1 (K), R73.2
- new net: C4.1, R72.1, R73.1, U5.6 (K), U5.8 (K)
- new net: D58.2 (A), R121.2
- new net: R35.2, SW4.2
- new net: C6.1, R85.1
- new net: JP14.1 (A), R124.1
- new net: D60.2 (A), D61.1 (K)
- new net: Q7.2 (G), R119.2
- new net: D27.2 (A), R53.1
- new net: JP32.2 (C), SW23.2
- new net: JP1.2 (C), SW6.2
- new net: D29.2 (A), D35.1 (K)
- new net: D54.2 (A), R108.2
- new net: Q5.1 (D), R67.2
- new net: Q6.2 (G), R70.2
- new net: D24.2 (A), D25.1 (K)
- new net: D18.1 (K), R113.2
- new net: Q9.2 (G), R140.1
- new net: D5.1 (K), Q3.1 (D)
- new net: D7.2 (A), D8.1 (K)
- new net 1V8_AON: D1.1 (K), D16.1 (K), D18.2 (A), D19.2 (A), D22.1 (K), D29.1 (K), D3.2 (A), D36.2 (A), D39.2 (A), D42.1 (K), D44.2 (A), D49.1 (K), D51.2 (A), D6.1 (K), D60.1 (K), D62.2 (A)
- new net 3V3: JP13.2 (B), JP18.2 (B), JP24.2 (B), JP27.2 (B), JP30.2 (B), JP36.2 (B), JP5.2 (B), JP7.2 (B), R106.1, R107.2, R118.1, R120.2, R132.1, R134.2, R21.2, R36.1, R38.1, R48.1, R74.1, R75.1, R78.1, R8.1, R80.1, R95.1, R98.2
- new net 3V3_AON: Q9.3 (S), R102.1, R103.1, R104.1, R105.1, R108.1, R109.2, R111.2, R114.1, R115.1, R116.1, R117.1, R121.1, R122.2, R124.2, R128.1, R129.1, R13.1, R130.1, R131.1, R135.1, R136.2, R138.2, R139.2, R14.1, R140.2, R15.1, R16.2, R22.1, R23.2, R25.2, R35.1, R39.2, R4.1, R42.1, R43.1, R44.1, R46.2, R5.1, R6.1, R7.1, R76.2, R77.1, R79.1, R81.1, R82.1, R83.2, R89.1, R90.1, R91.1, R92.2, R93.1, R96.2, R97.1
- new net VREF_EN: R27.2
- new net VSYS: D15.2 (A), D21.2 (A), D38.2 (A), D46.2 (A), D55.2 (A), D59.2 (A), D66.2 (A), R47.1, R84.1
- new net ~{PSRAM_CS}: R139.1
- new net ~{RESET}: JP1.3 (B), JP2.3 (B), JP32.3 (B), JP35.3 (B)
Other:
- note added: "0 free IO"
- note added: "1"
- note added: "1 free IOs"
- note added: "1.0V reg"
- note added: "1.8V"
- note added: "1.8V CMOS compatible EN for any VIN or VOUT"
- note added: "1.8V LVCMOS header"
- note added: "1.8V reg"
- note added: "11 free IOs"
- note added: "20-27"
- note added: "3 free IOs"
- note added: "3.3V"
- note added: "3.3V AON"
- note added: "3.3V reg"
- note added: "36-39"
- note added: "36-40"
- note added: "3V"
- note added: "4 free IOs"
- note added: "40-41"
- note added: "42-46"
- note added: "44-45"
- note added: "7"
- note added: "8 single ended or 4 differential"
- note added: "9-11"
- note added: "AD"
- note added: "ADC_AVDD"
- note added: "Analog header"
- note added: "Analog switch"
- note added: "CC"
- note added: "CSI FPC"
- note added: "D+ & D-"
- note added: "DNF"
- note added: "DONE 11"
- note added: "DONE 7"
- note added: "DSI FPC"
- note added: "Device"
- note added: "Differential input pairs"
- note added: "EN"
- note added: "FPGA EN 46"
- note added: "FPGA_EN 39"
- note added: "FPGA_EN 46"
- note added: "Fixed 3.3V IOVDD PMODs are on same edge of board"
- note added: "HSTX 12-19"
- note added: "Host"
- note added: "I2C"
- note added: "I2C LED driver"
- note added: "I2C LED driver LP5810"
- note added: "I2C header"
- note added: "I2C header / Stemma QT"
- note added: "I2C0 0-1"
- note added: "I2C0 4-5"
- note added: "I2C1"
- note added: "I2C1 & ~{IRQ} 2-4"
- note added: "I2C1 2-3"
- note added: "IO Expander AW9523"
- note added: "JTAG_EN 10"
- note added: "JTAG_EN 8"
- note added: "LED / button connector"
- note added: "LED 6-8"
- note added: "LED cannot turn on while DONE outputs low. When DONE is hi-z, RP can control LED."
- note added: "LED header"
- note added: "Multi-function"
- note added: "Multi-function 38"
- note added: "Multi-function 5"
- note added: "NX bank 1 11 IOs total 3.3V Hot socketing"
- note added: "OSC_EN 9"
- note added: "Open drain"
- note added: "PROGRAM 4"
- note added: "PSRAM 3.3V"
- note added: "QMI_CS1 0"
- note added: "QMI_CS1 47"
- note added: "RP bank 0 48 IOs total IOVDD 1.8V 3.3V tolerant"
- note added: "RP bank 1 QSPI_IOVDD, USB_OTP_VDD 3.3V"
- note added: "Repeated for other FPGA power domains"
- note added: "SCL"
- note added: "SDA"
- note added: "SPI"
- note added: "SPI PMOD"
- note added: "SPI config"
- note added: "SPI config port"
- note added: "SWD header / JST"
- note added: "Shared LED 6"
- note added: "Shared PMOD 20-27"
- note added: "Shared PMOD 28-35"
- note added: "Shared PMOD 36-43"
- note added: "Shared button 5"
- note added: "USB device"
- note added: "USB device/host config & USB boot same as pico2-ice"
- note added: "USB port"
- note added: "VCC"
- note added: "VSYS"
- note added: "XIN/XOUT"
- note added: "device"
- note added: "host"
- note added: "x2"
- note added: "~{FPGA_EN} 46"
- note added: "~{I2C_IRQ}"
- note added: "~{I2C_IRQ} 1"
- note added: "~{I2C_IRQ} 10"
- note added: "~{I2C_IRQ} 4"
- note added: "~{JTAG_EN} 8"
- note added: "~{PROGRAM} 4"
- note added: "~{QMI_CS1} 47"
- note added: "~{RESET}"
- note added: "~{VREF_EN}"
- note removed: "1.8V SWD header"
- note removed: "16"
- note removed: "4 lanes"
- note removed: "8 data lanes, 2 clock lanes"
- note removed: "CLOCK GPIN"
- note removed: "HSTX"
- note removed: "High speed connector(s)"
- note removed: "Master SPI config port"
- note removed: "Output compensation resistor network"
- note removed: "RP Bank 0 48 IOs total IOVDD 1.8V 3.3V tolerant"
- note removed: "RP Bank 1 IOVDD 3.3V"
- note removed: "RP PMOD"
- note removed: "Shared I2C"
- note removed: "Shared PMOD 1"
- note removed: "Shared PMOD 2"
- note removed: "Shared btn"
- note removed: "diff input pairs"
- note removed: "~{QMI_CS1}"
