File: board/Rev0/pico2-nx/Connectors.kicad_sch (KiCad schematic)
At the start: 2 parts, among them J3 Conn_02x20_Odd_Even, J4 Conn_02x20_Odd_Even

Commit message: draft rev 0 work in progress
Parts:
- removed J3, J4: Conn_02x20_Odd_Even, symbol Connector_Generic:Conn_02x20_Odd_Even
- added C50: 4.7u, Capacitor_SMD:C_0402_1005Metric, symbol Device:C
- added C76, C77, C78, C79, C80: 0.1u, Capacitor_SMD:C_0201_0603Metric, symbol Device:C
- added D10: PRTR5V0U2X, Package_TO_SOT_SMD:SOT-143, symbol Power_Protection:PRTR5V0U2X
- added D2: 1N5819WS, Diode_SMD:D_SOD-323, symbol Device:D_Schottky
- added J1: USB_C_Receptacle_USB2.0, Connector_USB:USB_C_Receptacle_HRO_TYPE-C-31-M-12, symbol Connector:USB_C_Receptacle_USB2.0
- added J3: ~, symbol Connector_Generic_MountingPin:Conn_01x22_MountingPin
- added J4: SFV22R-2STE1HLF, RP2350_60QFN_minimal:AMPHENOL_SFV22R-2STE1HLF, symbol Connector_Generic_MountingPin:Conn_01x22_MountingPin
- added J5, J8: Conn_02x18_Odd_Even, symbol Connector_Generic:Conn_02x18_Odd_Even
- added J6: Conn_01x15, symbol Connector_Generic:Conn_01x15
- added J7, J9: SM04B-SRSS-TB, Connector_JST:JST_SH_SM04B-SRSS-TB_1x04-1MP_P1.00mm_Horizontal, symbol Connector_Generic_MountingPin:Conn_01x04_MountingPin
- added JP1, JP2, JP7: SolderJumper_3_Bridged12, Jumper:SolderJumper-3_P1.3mm_Bridged12_RoundedPad1.0x1.5mm, symbol Jumper:SolderJumper_3_Bridged12
- added JP5, JP6: SolderJumper_2_Open, Jumper:SolderJumper-2_P1.3mm_Open_RoundedPad1.0x1.5mm, symbol Jumper:SolderJumper_2_Open
- added PTC1: MF-FSMF035X-2, Resistor_SMD:R_0603_1608Metric, symbol Device:R
- added R36, R38: 56K, Resistor_SMD:R_0402_1005Metric, symbol Device:R
- added R37, R39: 5.1K, Resistor_SMD:R_0402_1005Metric, symbol Device:R
- added R61, R64, R65, R66, R67: 200K, Resistor_SMD:R_0402_1005Metric, symbol Device:R
- added R68, R69: 200, Resistor_SMD:R_0402_1005Metric, symbol Device:R
- added R73, R74: 200, Resistor_SMD:R_0402_1005Metric, symbol Device:R_Small
- added U14: 74LV4066, Package_SO:SO-14_3.9x8.65mm_P1.27mm, symbol Analog_Switch:CD4066BM
- added U15, U16: TXS0108EPW, Package_SO:TSSOP-20_4.4x6.5mm_P0.65mm, symbol Logic_LevelTranslator:TXS0108EPW
Connections:
- new net: D2.1 (K), PTC1.2
- new net: JP1.1 (A), R37.1
- new net: J1.B5 (CC2), JP1.2 (C)
- new net: JP1.3 (B), R36.2
- new net: JP6.2 (B), R74.1
- new net: JP2.1 (A), R39.1
- new net: J1.A5 (CC1), JP2.2 (C)
- new net: JP2.3 (B), R38.2
- new net: JP5.2 (B), R73.1
- new net ADC0: R68.1
- new net ADC0_PROT: D10.3 (I/O2), J8.27 (Pin_27), R68.2
- new net ADC1: R69.1
- new net ADC1_PROT: D10.2 (I/O1), J8.28 (Pin_28), R69.2
- new net DONE: J8.34 (Pin_34)
- new net EXT_LED: J5.17 (Pin_17)
- new net EXT_MIPI.CLK+: J3.14 (Pin_14)
- new net EXT_MIPI.CLK-: J3.15 (Pin_15)
- new net EXT_MIPI.D0+: J3.20 (Pin_20)
- new net EXT_MIPI.D0-: J3.21 (Pin_21)
- new net EXT_MIPI.D1+: J3.17 (Pin_17)
- new net EXT_MIPI.D1-: J3.18 (Pin_18)
- new net EXT_MIPI.D2+: J3.11 (Pin_11)
- new net EXT_MIPI.D2-: J3.12 (Pin_12)
- new net EXT_MIPI.D3+: J3.8 (Pin_8)
- new net EXT_MIPI.D3-: J3.9 (Pin_9)
- new net EXT_SPI.CSn: J6.1 (Pin_1)
- new net EXT_SPI.MISO: J6.3 (Pin_3), JP6.1 (A)
- new net EXT_SPI.MOSI: J6.2 (Pin_2), JP5.1 (A)
- new net EXT_SPI.SCK: J6.4 (Pin_4)
- new net FPC_IO.LED_EN: J3.5 (Pin_5), J4.18 (Pin_18)
- new net FPC_IO.PWR_EN: J3.6 (Pin_6), J4.17 (Pin_17)
- new net FPGA_CLK_EN: J8.24 (Pin_24)
- new net FPGA_EN: J8.23 (Pin_23), U14.12, U14.13, U14.5, U14.6
- new net FPGA_PMOD0: J8.22 (Pin_22)
- new net FPGA_PMOD1: J8.20 (Pin_20)
- new net FPGA_PMOD2: J8.18 (Pin_18)
- new net FPGA_PMOD3: J8.16 (Pin_16)
- new net FPGA_PMOD4: J8.21 (Pin_21)
- new net FPGA_PMOD5: J8.19 (Pin_19)
- new net FPGA_PMOD6: J8.17 (Pin_17)
- new net FPGA_PMOD7: J8.15 (Pin_15)
- new net GND: C50.2, C76.2, C77.2, C78.2, C79.2, C80.2, D10.1 (GND), J1.A1 (GND), J1.A12 (GND), J1.B1 (GND), J1.B12 (GND), J1.S1 (SHIELD), J3.10 (Pin_10), J3.13 (Pin_13), J3.16 (Pin_16), J3.19 (Pin_19), J3.22 (Pin_22), J3.4 (Pin_4), J3.7 (Pin_7), J3.MP (MountPin), J4.1 (Pin_1), J4.10 (Pin_10), J4.13 (Pin_13), J4.16 (Pin_16), J4.19 (Pin_19), J4.4 (Pin_4), J4.7 (Pin_7), J4.MP (MountPin), J5.13 (Pin_13), J5.14 (Pin_14), J5.20 (Pin_20), J5.31 (Pin_31), J5.32 (Pin_32), J5.36 (Pin_36), J5.4 (Pin_4), J6.14 (Pin_14), J6.5 (Pin_5), J7.4 (Pin_4), J7.MP (MountPin), J8.13 (Pin_13), J8.14 (Pin_14), J8.25 (Pin_25), J8.3 (Pin_3), J8.31 (Pin_31), J8.5 (Pin_5), J9.4 (Pin_4), J9.MP (MountPin), R37.2, R39.2, R61.2, U14.7 (V_{SS}), U15.11 (GND), U16.11 (GND)
- new net I2C0.SCL: J5.21 (Pin_21), J9.1 (Pin_1), U14.4
- new net I2C0.SDA: J5.22 (Pin_22), J9.2 (Pin_2), U14.11
- new net I2C1.SCL: J7.1 (Pin_1), J8.30 (Pin_30), U14.1
- new net I2C1.SDA: J7.2 (Pin_2), J8.29 (Pin_29), U14.8
- new net I2C_IRQn: J5.19 (Pin_19), J8.32 (Pin_32)
- new net LED.B: J6.9 (Pin_9)
- new net LED.G: J6.8 (Pin_8)
- new net LED.MONO: J5.18 (Pin_18)
- new net LED.R: J6.7 (Pin_7)
- new net MULTI_FN: J8.33 (Pin_33)
- new net P1V8D: D10.4 (VCC)
- new net P1V8D_FPGA: C77.1, C78.1, U15.2 (VCCA), U16.2 (VCCA)
- new net P3V3A_VREF: J5.3 (Pin_3)
- new net P3V3D: C76.1, U14.14 (V_{DD})
- new net P3V3D_FPGA: C79.1, J3.1 (Pin_1), J4.22 (Pin_22), J5.15 (Pin_15), J5.16 (Pin_16), J6.15 (Pin_15), J6.6 (Pin_6), J7.3 (Pin_3), J8.1 (Pin_1), J8.11 (Pin_11), J8.12 (Pin_12), J9.3 (Pin_3), JP7.1 (A), R64.1, R65.1, R66.1, R67.1, U15.19 (VCCB)
- new net P5VD: C50.1, J5.2 (Pin_2), PTC1.1
- new net P5VD_VBUS: D2.2 (A), J1.A4 (VBUS), J1.A9 (VBUS), J1.B4 (VBUS), J1.B9 (VBUS), J5.1 (Pin_1), R36.1, R38.1
- new net PxVD_SBIN: J5.35 (Pin_35), JP7.3 (B)
- new net PxVD_SBOUT: C80.1, J5.33 (Pin_33), J5.34 (Pin_34), JP7.2 (C), U16.19 (VCCB)
- new net RESETn: J8.36 (Pin_36)
- new net RGB_MIPI.CLK+: J4.9 (Pin_9)
- new net RGB_MIPI.CLK-: J4.8 (Pin_8)
- new net RGB_MIPI.D0+: J4.3 (Pin_3)
- new net RGB_MIPI.D0-: J4.2 (Pin_2)
- new net RGB_MIPI.D1+: J4.6 (Pin_6)
- new net RGB_MIPI.D1-: J4.5 (Pin_5)
- new net RGB_MIPI.D2+: J4.12 (Pin_12)
- new net RGB_MIPI.D2-: J4.11 (Pin_11)
- new net RGB_MIPI.D3+: J4.15 (Pin_15)
- new net RGB_MIPI.D3-: J4.14 (Pin_14)
- new net RP_SPI.CSn: J6.10 (Pin_10)
- new net RP_SPI.MISO: J6.12 (Pin_12)
- new net RP_SPI.MOSI: J6.11 (Pin_11)
- new net RP_SPI.SCK: J6.13 (Pin_13)
- new net SCL0: J3.3 (Pin_3), R65.2, U14.3
- new net SCL1: J4.20 (Pin_20), R64.2, U14.2
- new net SDA0: J3.2 (Pin_2), R67.2, U14.10
- new net SDA1: J4.21 (Pin_21), R66.2, U14.9
- new net SHARED_A0: J5.5 (Pin_5), U15.20 (B1)
- new net SHARED_A1: J5.7 (Pin_7), U15.18 (B2)
- new net SHARED_A2: J5.9 (Pin_9), U15.17 (B3)
- new net SHARED_A3: J5.11 (Pin_11), U15.16 (B4)
- new net SHARED_A4: J5.6 (Pin_6), U15.15 (B5)
- new net SHARED_A5: J5.8 (Pin_8), U15.14 (B6)
- new net SHARED_A6: J5.10 (Pin_10), U15.13 (B7)
- new net SHARED_A7: J5.12 (Pin_12), U15.12 (B8)
- new net SHARED_B0: J5.23 (Pin_23), U16.20 (B1)
- new net SHARED_B1: J5.25 (Pin_25), U16.18 (B2)
- new net SHARED_B2: J5.27 (Pin_27), U16.17 (B3)
- new net SHARED_B3: J5.29 (Pin_29), U16.16 (B4)
- new net SHARED_B4: J5.24 (Pin_24), U16.15 (B5)
- new net SHARED_B5: J5.26 (Pin_26), U16.14 (B6)
- new net SHARED_B6: J5.28 (Pin_28), U16.13 (B7)
- new net SHARED_B7: J5.30 (Pin_30), U16.12 (B8)
- new net SHARED_PMOD_A0: U15.1 (A1)
- new net SHARED_PMOD_A1: U15.3 (A2)
- new net SHARED_PMOD_A2: U15.4 (A3)
- new net SHARED_PMOD_A3: U15.5 (A4)
- new net SHARED_PMOD_A4: U15.6 (A5)
- new net SHARED_PMOD_A5: U15.7 (A6)
- new net SHARED_PMOD_A6: U15.8 (A7)
- new net SHARED_PMOD_A7: U15.9 (A8)
- new net SHARED_PMOD_B0: U16.1 (A1)
- new net SHARED_PMOD_B1: U16.3 (A2)
- new net SHARED_PMOD_B2: U16.4 (A3)
- new net SHARED_PMOD_B3: U16.5 (A4)
- new net SHARED_PMOD_B4: U16.6 (A5)
- new net SHARED_PMOD_B5: U16.7 (A6)
- new net SHARED_PMOD_B6: U16.8 (A7)
- new net SHARED_PMOD_B7: U16.9 (A8)
- new net SHARED_PMOD_EN: J8.26 (Pin_26), R61.1, U15.10 (OE), U16.10 (OE)
- new net UJTAG.PRESENTn: J8.10 (Pin_10)
- new net UJTAG.TCK: J8.4 (Pin_4)
- new net UJTAG.TDI: J8.8 (Pin_8)
- new net UJTAG.TDO: J8.6 (Pin_6)
- new net UJTAG.TMS: J8.2 (Pin_2)
- new net UJTAG_RXD: J8.9 (Pin_9), R74.2
- new net UJTAG_TXD: J8.7 (Pin_7), R73.2
- new net USB.D+: J1.A6 (D+), J1.B6 (D+)
- new net USB.D-: J1.A7 (D-), J1.B7 (D-)
- new net USB_BOOTn: J8.35 (Pin_35)
- no-connect marks 0 -> 2
Other:
- note added: "All 100 mil pitch headers a multiple of 100 mils apart on pin centers, so footprint is easy to replicate"
- note added: "All connectors, LEDs and buttons on top."
- note added: "Peripheral(Default)/Host Selection Host Mode: Solder open bridges, cut shorted bridges Peripheral: Default"
- note added: "TODO: Should TXD & RXD be swapped?"
- note added: "USBC Connector"
- note added: "https://github.com/tinyvision-ai-inc/upduino-jtag"
