File: board/Rev0/pico2-nx/FPGA.kicad_sch (KiCad schematic)
At the start: 73 parts, among them T1 TP_S, U1 LIFCL-17-CSFBGA121, U2 W25Q32JVSSIQ, U3 S27KS0641DPBHI020, U4 LIFCL-17-7MG121C, U5 LIFCL-17-CSFBGA121, Y1 DSC6001ME2A-024.0000

Commit message: draft rev 0 work in progress
Parts:
- removed C1, C10, C12, C16, C18, C2, C20, C21, C22, C23, C3, C30, C31, C32, C33, C8: 10uF, CAPC1005X55USR, symbol pico2-nx-altium-import:root_1_Cap_1uF_X5R_10%_6V3_0402
- removed C11, C13, C14, C15, C24, C25, C26, C27, C28, C29, C34, C36, C37, C38, C39, C4, C40, C41, C5, C6, C7, C9: ${ALTIUM_VALUE}, CAPC0603X33N, symbol pico2-nx-altium-import:root_1_CAP CER 0.1UF 10V X7S 0201
- removed C17, C19: ${ALTIUM_VALUE}, CAPC0603X33N, symbol pico2-nx-altium-import:root_1_CAP CER 4.7UF 6.3V X5R 0201
- removed C35: ${ALTIUM_VALUE}, CAPC0603X33N, symbol pico2-nx-altium-import:root_2_CAP CER 0.1UF 10V X7S 0201
- removed R1, R11, R12, R13, R14, R15, R2, R3, R4, R8, R9: 10K, RESC0603X26N, symbol pico2-nx-altium-import:root_0_mirrored_Res_10K_1%_0402
- removed R10, R7: ${ALTIUM_VALUE}, RESC0603X26N, symbol pico2-nx-altium-import:root_2_mirrored_RES 4.7K OHM 1% 1/20W 0201
- removed R17: ${ALTIUM_VALUE}, RESC0603X26N, symbol pico2-nx-altium-import:root_0_mirrored_Res_10K_1%_0402
- removed R27: ${ALTIUM_VALUE}, RESC0603X26N, symbol pico2-nx-altium-import:root_1_mirrored_Res_10K_1%_0402
- removed R5, R6: ${ALTIUM_VALUE}, RESC0603X26N, symbol pico2-nx-altium-import:root_2_mirrored_Res_10K_1%_0402
- removed T1: TP_S, TP 1mm, symbol pico2-nx-altium-import:root_2_TP_S_0
- removed Y1: DSC6001ME2A-024.0000, XTAL_20X16X09, symbol pico2-nx-altium-import:root_0_AMPMAFB-24.0000T
- added C10, C15, C18, C23, C24, C25, C27, C28, C29, C30, C35, C36, C39, C40, C7, C8, C83, C84, C9: 10u, Capacitor_SMD:C_0402_1005Metric, symbol Device:C
- added C11, C12, C13, C14, C16, C17, C19, C20, C21, C22, C31, C32, C33, C34, C37, C38, C41, C42, C43, C44, C45, C46, C47, C85: 0.1u, Capacitor_SMD:C_0201_0603Metric, symbol Device:C
- added C26: 4.7u, Capacitor_SMD:C_0402_1005Metric, symbol Device:C
- added C81: 1u, Capacitor_SMD:C_0402_1005Metric, symbol Device:C
- added D6: 1N5819WS, Diode_SMD:D_SOD-323, symbol Device:D_Schottky
- added Q1: BSS84, Package_TO_SOT_SMD:SOT-23, symbol Transistor_FET:BSS84
- added R10, R13, R15, R16, R59, R9: 4.7K, Resistor_SMD:R_0402_1005Metric, symbol Device:R_Small
- added R11: 2.2K, Resistor_SMD:R_0402_1005Metric, symbol Device:R_Small
- added R12, R28, R29, R30, R31, R32, R62: 10K, Resistor_SMD:R_0402_1005Metric, symbol Device:R_Small
- added R27: 27, Resistor_SMD:R_0402_1005Metric, symbol Device:R_Small
- added R33: 22, Resistor_SMD:R_0402_1005Metric, symbol Device:R_Small
- added R72: 0, Resistor_SMD:R_0402_1005Metric, symbol Device:R_Small
- added U17: SN74CB3Q3257, symbol 74xx:74CBTLV3257
- added Y1: SG-210STF 24.0000ML0, Oscillator:Oscillator_SMD_SeikoEpson_SG210-4Pin_2.5x2.0mm, symbol Oscillator:SG-210STF
- FB1, FB2, FB3, FB4, FB5, FB6, FB7, FB8: footprint 0402_FB -> (none); symbol pico2-nx-altium-import:root_0_MURA-FB-2 -> Device:L
- U3: renamed from U1; value LIFCL-17-CSFBGA121 -> LIFCL-17-7MG121C; footprint BGA121C50P11X11_600X600X100 -> (none)
- U3: renamed from U5; value LIFCL-17-CSFBGA121 -> LIFCL-17-7MG121C; footprint BGA121C50P11X11_600X600X100 -> (none)
- U3: renamed from U4; footprint BGA121C50P11X11_600X600X100 -> (none)
- U4: renamed from U2; value W25Q32JVSSIQ -> W25Q128JVSSIQ; MPN W25Q32JVSSIQ -> W25Q128JVSSIQ
- U5: renamed from U3; value S27KS0641DPBHI020 -> APS6408L-OBM-BA; footprint BGA24C100P5X5_800X600X120N -> (none); ARROW PART NUMBER S27KS0641DPBHI020 -> (none); ARROW PRICE/STOCK https://www.arrow.com/en/products/s27ks0641dpbhi020/cypress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 -> (none); DATASHEET LINK http://www.cypress.com/file/183506/download -> (none); DIGI-KEY PART NUMBER 428-3858-ND -> (none); MANUFACTURER Cypress Semiconductor -> (none); MANUFACTURER PRODUCT NUMBER S27KS0641DPBHI020 -> (none); MOUSER PRICE/STOCK https://www.mouser.co.uk/ProductDetail/Cypress-Semiconducto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 -> (none)
Connections:
- net DONE: now also R62.2
- net FPGA_CLK: now also U3.G4 (PB60A/PCLKT3_1/ADC_CP6), R33.2
- net FPGA_CLK_EN: now also Y1.1 (~{ST})
- net GND: now also C10.2, C11.2, C12.2, C13.2, C14.2, C15.2, C16.2, C17.2, C18.2, C19.1, C20.2, C21.2, C22.2, C23.2, C24.2, C25.2, C26.2, C27.2, C28.2, C29.1, C30.1, C31.2, C32.2, C33.2, C34.2, C35.2, C36.2, C37.1, C38.1, C39.2, C40.2, C41.2, C42.2, C43.2, C44.2, C45.2, C46.2, C47.2, C7.2, C8.2, C81.1, C83.2, C84.2, C85.1, C9.2, R11.2, R9.2, U17.15 (~{OE}), U17.8 (GND), Y1.2 (GND)
- net JTAG_EN: now also Q1.3 (D), R9.1
- net P1V8D_FPGA: now also C10.1, C13.1, C14.1, C15.1, C16.1, C18.1, C19.2, C20.1, C21.1, C22.1, C81.2, C83.1, C84.1, C9.1, R12.2, R31.2, R32.2, Y1.4 (Vcc)
- net P1VD_FPGA: now also C23.1, C28.1, C35.1, C41.1, C43.1, C45.1
- net P3V3D_FPGA: now also C11.1, C12.1, C17.1, C7.1, C8.1, C85.2, Q1.2 (S), R10.2, R13.1, R15.2, R16.2, R28.1, R29.2, R30.2, R59.1, R62.1, U17.16 (VCC)
- net PVCCAUX: now also C36.1, C40.1, C44.1, C46.1, C47.1
- net SRAM_CEN: now also U3.K5 (PB54B/PCLKC4_0/VREF4_2), R31.1; no longer U3.K1 (PB64A/ADC_CP8)
- net SRAM_CLK_N: now also U3.H7 (PB44B); no longer U3.J2 (PB66B/PCLKC3_2/ADC_CN13)
- net SRAM_CLK_P: now also U3.H8 (PB44A); no longer U3.J1 (PB66A/PCLKT3_2/ADC_CP13)
- net SRAM_DQ0: now also U3.G8 (PB46B); no longer U3.L4 (PB56A/PCLKT3_0/VREF3_1/ADC_CP5)
- net SRAM_DQ1: now also U3.F7 (PB48A/PCLKT4_2); no longer U3.L3 (PB56B/PCLKC3_0/ADC_CN5)
- net SRAM_DQ2: now also U3.F6 (PB48B/PCLKC4_2); no longer U3.J4 (PB58A/ADC_CP7)
- net SRAM_DQ3: now also U3.F5 (PB50A); no longer U3.K4 (PB58B/ADC_CN7)
- net SRAM_DQ4: now also U3.G5 (PB50B); no longer U3.G4 (PB60A/PCLKT3_1/ADC_CP6)
- net SRAM_DQ5: now also U3.H5 (PB52A/PCLKT4_1); no longer U3.H4 (PB60B/PCLKC3_1/ADC_CN6)
- net SRAM_DQ6: now also U3.J5 (PB52B/PCLKC4_1); no longer U3.L2 (PB62A/ADC_CP9)
- net SRAM_DQ7: now also U3.L5 (PB54A/PCLKT4_0); no longer U3.L1 (PB62B/ADC_CN9)
- net SRAM_RW: now also U3.G7 (PB46A); no longer U3.H1 (PB68A/PCLKT3_3/ADC_CP14)
- net TCK: now also R11.1, U17.12
- net TDI: now also R15.1, U17.7
- net TDO: now also R10.1, U17.9
- net TMS: now also R16.1, U17.4
- net at FB3.2, U3.C8 (VCCPLLDPHY0): now also C24.1, C31.1
- net at FB4.2, U3.D9 (VCCDPHY0): now also C25.1, C32.1
- net at FB1.2, U3.F10 (VCCADPHY0): now also C29.2, C37.2
- net at FB5.2, U3.C6 (VCCPLLDPHY1): now also C26.1, C33.1
- net at FB8.2, U3.G9 (VCCAUXH5): now also C39.1, C42.1
- net SHARED_PMOD_A7: now reaches U3.L7 (PB22A)
- net at FB2.2, U3.A4 (VCCADPHY1): now also C30.2, C38.2
- net at FB6.2, U3.C4 (VCCDPHY1): now also C27.1, C34.1
- net I2C1.SDA: now reaches U3.D1 (PR9B)
- net QSPI.SCLK: now reaches U3.E1 (PR11B/PCLKT1_2)
- net I2C1.SCL: now reaches U3.E2 (PR11A)
- net FPGA_PMOD7: now reaches U3.F1 (PR13B/PCLKT1_0)
- net FPGA_PMOD3: now reaches U3.F2 (PR13A/PCLKT1_1)
- net FPGA_PMOD1: now reaches U3.B3 (PT67A)
- net FPGA_PMOD5: now reaches U3.C3 (PT67B)
- net FPGA_PMOD4: now reaches U3.E3 (PT65B/MCSNO/MSDO)
- net SHARED_PMOD_A0: now reaches U3.G10 (PB16B/CDR_RXN0/ADC_CN0/COMP1N)
- net SHARED_PMOD_A2: now reaches U3.G11 (PB16A/CDR_RXP0/VREF5_1/ADC_CP0/COMP1P)
- net SHARED_PMOD_A1: now reaches U3.H10 (PB18B/PCLKC5_0/CDR_RXN1/ADC_CN1/COMP2N)
- net SHARED_PMOD_A3: now reaches U3.H11 (PB18A/PCLKT5_0/CDR_RXP1/ADC_CP1/COMP2P)
- net SHARED_PMOD_A6: now reaches U3.J10 (PB20B/PCLKC5_1/LLC_GPLL0C_IN/ADC_CN3)
- net SHARED_PMOD_A4: now reaches U3.J11 (PB20A/PCLKT5_1/LLC_GPLL0T_IN/ADC_CP3)
- net SHARED_PMOD_B6: now reaches U3.J7 (PB28B)
- net SHARED_PMOD_B5: now reaches U3.K10 (PB30B/PCLKC5_3/VREF5_2)
- net SHARED_PMOD_B3: now reaches U3.K11 (PB26A/PCLKT5_2/ADC_CP2/COMP3P)
- net SHARED_PMOD_B0: now reaches U3.K6 (PB24B)
- net SHARED_PMOD_B4: now reaches U3.K7 (PB28A)
- net SHARED_PMOD_B7: now reaches U3.L10 (PB30A/PCLKT5_3)
- net SHARED_PMOD_B1: now reaches U3.L11 (PB26B/PCLKC5_2/ADC_CN2/COMP3N)
- net SHARED_PMOD_B2: now reaches U3.L6 (PB24A)
- net SHARED_PMOD_A5: now reaches U3.L8 (PB22B)
- net HSTX7: now reaches U3.G1 (PB70B/LRC_GPLL0C_IN/VREF3_2)
- net HSTX6: now reaches U3.G2 (PB70A/LRC_GPLL0T_IN)
- net HSTX5: now reaches U3.H2 (PB68B/PCLKC3_3/ADC_CN14)
- net EXT_MIPI_CLK_N renamed EXT_MIPI.CLK-
- net EXT_MIPI_CLK_P renamed EXT_MIPI.CLK+
- net EXT_MIPI_D0_N renamed EXT_MIPI.D0-
- net EXT_MIPI_D0_P renamed EXT_MIPI.D0+
- net EXT_MIPI_D1_N renamed EXT_MIPI.D1-
- net EXT_MIPI_D1_P renamed EXT_MIPI.D1+
- net EXT_MIPI_D2_N renamed EXT_MIPI.D2-
- net EXT_MIPI_D2_P renamed EXT_MIPI.D2+
- net EXT_MIPI_D3_N renamed EXT_MIPI.D3-
- net EXT_MIPI_D3_P renamed EXT_MIPI.D3+
- net FFLASH_SCK: no longer names the net of U3.E7 (PT59A/MCLK/PCLKT0_0)
- net FFLASH_SCK: now also R27.1; no longer U4.6 (CLK)
- net FFLASH_SIO0 renamed EXT_SPI.MOSI
- net FFLASH_SIO1 renamed EXT_SPI.MISO
- net FFLASH_SIO2: no longer names the net of U4.3 (IO2)
- net FFLASH_SIO2: now also R29.1; no longer U3.D5 (PT63B/MD2)
- net FFLASH_SIO3: no longer names the net of U4.7 (IO3)
- net FFLASH_SIO3: now also R30.1; no longer U3.E4 (PT65A/MD3)
- net FFLASH_SSN renamed FLASH_CSn
- net FLASH_CSn: now also R28.2
- net INITn renamed EXT_SPI.CSn
- net PROGn renamed MULTI_FN
- net RGB_MIPI_CLK_N renamed RGB_MIPI.CLK-
- net RGB_MIPI_CLK_P renamed RGB_MIPI.CLK+
- net RGB_MIPI_D0_N renamed RGB_MIPI.D0-
- net RGB_MIPI_D0_P renamed RGB_MIPI.D0+
- net RGB_MIPI_D1_N renamed RGB_MIPI.D1-
- net RGB_MIPI_D1_P renamed RGB_MIPI.D1+
- net RGB_MIPI_D2_N renamed RGB_MIPI.D2-
- net RGB_MIPI_D2_P renamed RGB_MIPI.D2+
- net RGB_MIPI_D3_N renamed RGB_MIPI.D3-
- net RGB_MIPI_D3_P renamed RGB_MIPI.D3+
- net SCL renamed FPGA_PMOD6
- net SDA renamed FPGA_PMOD2
- net SRAM_RSTN renamed HSTX1
- net HSTX1: no longer U5.A4 (RESET#)
- new net: R33.1, Y1.3 (OUT)
- new net: R72.1, U17.14
- new net EXT_SPI.SCK: R27.2, U4.6 (CLK)
- new net FPC_IO_1V8.LED_EN: U3.J4 (PB58A/ADC_CP7)
- new net FPC_IO_1V8.PWR_EN: U3.L3 (PB56B/PCLKC3_0/ADC_CN5)
- new net FPGA_PMOD0: U3.E4 (PT65A/MD3)
- new net HSTX0: U3.K1 (PB64A/ADC_CP8)
- new net HSTX2: U3.J1 (PB66A/PCLKT3_2/ADC_CP13)
- new net HSTX3: U3.J2 (PB66B/PCLKC3_2/ADC_CN13)
- new net HSTX4: U3.H1 (PB68A/PCLKT3_3/ADC_CP14)
- new net I2C_IRQn: U3.D5 (PT63B/MD2)
- new net JTAG_ENn: D6.2 (A), Q1.1 (G), R59.2
- new net QSPI.CSn: R12.1, U3.L4 (PB56A/PCLKT3_0/VREF3_1/ADC_CP5)
- new net QSPI.SD0: U17.3
- new net QSPI.SD1: U17.6
- new net QSPI.SD2: U17.10
- new net QSPI.SD3: U17.13
- new net SRAM_RSTn: R32.1, U5.A4 (RESET#)
- new net UJTAG.PRESENTn: D6.1 (K), R13.2, U17.1 (S)
- new net UJTAG.TCK: R72.2
- new net UJTAG.TDI: U17.5
- new net UJTAG.TDO: U17.11
- new net UJTAG.TMS: U17.2
- no-connect marks 4 -> 13
Other:
- note added: "CK# HyperRAM only"
- note added: "DQS"
- note added: "FPGA Flash"
- note added: "Hot socketing I_{OFF} < 1uA"
- note added: "QSPI bus is also used for JTAG"
- note added: "RP CLK GPOUT3"
- note added: "RP SPI0 SCLK"
- note added: "RP SPI1 SCLK"
- note added: "Route as differential pairs, HSTX0/HSTX1, 2/3, 4/5, 6/7."
- note added: "TODO: checklist recommends a resistor between power supply and oscillator VDD."
- note added: "Unlike other QSPI nets, which are 3.3V CMOS level, CSn is 1.8V CMOS level."
- note added: "Upduino JTAG"
- note added: "Xcella RAM"
- note removed: "HyperRAM"
- note removed: "I2C and JTAG Pullups"
- moved on the sheet: U3A, U3B, U3C, U3D, U3E, U3F, U3G, U3H, U3I, U4, U5
