File: board/Rev0/pico2-nx/Power.kicad_sch (KiCad schematic)
At the start: 28 parts, among them T1 3V3, T2 1V0, T22 3V3, U6 TPS22917DBV

Commit message: draft rev 0 work in progress
Parts:
- removed C33, C34, C35, C36, C4: ${ALTIUM_VALUE}, CAP_0603, symbol pico2-nx-altium-import:root_1_Cap_1uF_X5R_10%_6V3_0402
- removed C37: ${ALTIUM_VALUE}, CAP_0603, symbol pico2-nx-altium-import:root_1_mirrored_Cap_1uF_X5R_10%_6V3_0402
- removed R12, R22, R25, R28, R31, R32: ${ALTIUM_VALUE}, RESC1005X40USR, symbol pico2-nx-altium-import:root_1_mirrored_Res_10K_1%_0402
- removed R21, R24, R30: ${ALTIUM_VALUE}, RESC1005X40USR, symbol pico2-nx-altium-import:root_0_mirrored_RES 0 OHM JUMPER 1/20W 0201
- removed R23: 100K, RESC1005X40USR, symbol pico2-nx-altium-import:root_1_mirrored_Res_10K_1%_0402
- removed R26: 294K, RESC1005X40USR, symbol pico2-nx-altium-import:root_1_mirrored_Res_10K_1%_0402
- removed U6: TPS22917DBV, Package_TO_SOT_SMD:SOT-23-6, symbol Power_Management:TPS22917DBV
- added C1, C2, C3, C4, C5, C6, C75, C82: 10u, Capacitor_SMD:C_0402_1005Metric, symbol Device:C
- added JP8: SolderJumper_2_Bridged, Jumper:SolderJumper-2_P1.3mm_Bridged_RoundedPad1.0x1.5mm, symbol Jumper:SolderJumper_2_Bridged
- added R18, R19, R20: 0, Resistor_SMD:R_0402_1005Metric, symbol Device:R_Small
- added R21, R23, R25, R75: 200K, Resistor_SMD:R_0402_1005Metric, symbol Device:R_Small
- added R22: 100K, Resistor_SMD:R_0402_1005Metric, symbol Device:R_Small
- added R24: 44.2K, Resistor_SMD:R_0402_1005Metric, symbol Device:R_Small
- added R26: 294K, Resistor_SMD:R_0402_1005Metric, symbol Device:R_Small
- added SJ3, SJ4: SHORT, Jumper:SolderJumper-2_P1.3mm_Bridged_RoundedPad1.0x1.5mm, symbol Device:R
- added TP5, TP6: TestPoint, symbol Connector:TestPoint
- added U1, U2: MIC2005A-2YM5-TR, symbol SamacSys:MIC2005A-2YM5-TR
- L1, L2, L3: value ${ALTIUM_VALUE} -> 1u; footprint INDC2016X100N -> (none); symbol pico2-nx-altium-import:root_0_725321dda6339637d4d059423bc1c3c -> Device:L
- PS1, PS2, PS3: footprint SOTFL50P160X60-6N -> (none)
- SJ1: symbol UPduino_v3.0:Device_R -> Device:R
- TP1: renamed from T1; value 3V3 -> 1V8; footprint TP 1mm -> (none); symbol pico2-nx-altium-import:root_3_TP_S_0 -> Connector:TestPoint
- TP2: renamed from T22; footprint TP 1mm -> (none); symbol pico2-nx-altium-import:root_3_TP_S_0 -> Connector:TestPoint
- TP3: renamed from T2; footprint TP 1mm -> (none); symbol pico2-nx-altium-import:root_3_TP_S_0 -> Connector:TestPoint
Connections:
- net FPGA_EN: now also U1.3 (ENABLE), U2.3 (ENABLE)
- net GND: now also C1.2, C2.2, C3.2, C4.2, C5.2, C6.2, C75.2, C82.2, R22.1, R24.1, R26.1, U1.2 (GND), U2.2 (GND)
- net P1V8D: now also C5.1, C82.1, R19.2, R21.2, SJ4.2
- net P1V8D_FPGA: now also U1.5 (VOUT)
- net P1VD_FPGA: now also R25.2, SJ3.1; no longer L2.2, TP3.1
- net P3V3D: now also C6.1, R20.2, R23.2
- net P3V3D_FPGA: now also U2.5 (VOUT); no longer SJ1.1
- net PWR_EN: now also JP8.1 (A)
- net at PS3.6 (OUT): now also R20.1
- net at PS2.1 (FB): now also R25.1, R26.2
- net at PS2.6 (OUT): now also R18.1
- net at PS1.1 (FB): now also R21.1, R22.2
- net at PS1.6 (OUT): now also R19.1
- net at PS3.1 (FB): now also R23.1, R24.2
- net V_{in} renamed P5VD
- net P5VD: now also C1.1, C2.1, C3.1, R75.2
- new net: SJ1.1, U2.1 (VIN)
- new net: C4.1, C75.1, L2.2, R18.2, SJ3.2, TP3.1
- new net: JP8.2 (B), R75.1
- new net: TP5.1, U2.4 (FAULT/)
- new net: SJ4.1, U1.1 (VIN)
- new net: TP6.1, U1.4 (FAULT/)
Other:
- moved on the sheet: PS1, PS2, PS3, SJ1
