File: board/Rev0/pico2-nx/RP2350.kicad_sch (KiCad schematic)
At the start: 62 parts, among them J1 BM03B-SRSS-TB, J2 USB_C_Receptacle_USB2.0, SW1 CS1213AGF260, U1 W25Q32JVSSIQ, U2 RP2350_80QFN, U3 TL431DBZ, Y1 ABM8-272-T3

Commit message: draft rev 0 work in progress
Parts:
- removed C13, C42: 4.7u, Capacitor_SMD:C_0402_1005Metric, symbol UPduino_v3.0:Device_C
- removed C16, C21: 0.1u, Capacitor_SMD:C_0402_1005Metric, symbol UPduino_v3.0:Device_C
- removed D3: 1N5819WS, Diode_SMD:D_SOD-323, symbol Device:D_Schottky
- removed J1: BM03B-SRSS-TB, Connector_JST:JST_SH_BM03B-SRSS-TB_1x03-1MP_P1.00mm_Vertical, symbol Connector_Generic_MountingPin:Conn_01x03_MountingPin
- removed J2: USB_C_Receptacle_USB2.0, Connector_USB:USB_C_Receptacle_HRO_TYPE-C-31-M-12, symbol Connector:USB_C_Receptacle_USB2.0
- removed JP1, JP2: SolderJumper_3_Bridged12, Jumper:SolderJumper-3_P1.3mm_Bridged12_RoundedPad1.0x1.5mm, symbol Jumper:SolderJumper_3_Bridged12
- removed PTC1: MF-FSMF035X-2, Resistor_SMD:R_0603_1608Metric, symbol UPduino_v3.0:Device_R
- removed R10, R14, R15: 27, Resistor_SMD:R_0402_1005Metric, symbol Device:R
- removed R11: 100, Resistor_SMD:R_0402_1005Metric, symbol UPduino_v3.0:Device_R
- removed R16, R17, R18: 10K, Resistor_SMD:R_0402_1005Metric, symbol Device:R
- removed R19, R20: SHORT, Jumper:SolderJumper-2_P1.3mm_Bridged_RoundedPad1.0x1.5mm, symbol Device:R
- removed R21: 1K, Resistor_SMD:R_0402_1005Metric, symbol Device:R
- removed R22, R24: 56K, Resistor_SMD:R_0402_1005Metric, symbol UPduino_v3.0:Device_R
- removed R23, R25: 5.1K, Resistor_SMD:R_0402_1005Metric, symbol UPduino_v3.0:Device_R
- removed R4: 10K, Resistor_SMD:R_0402_1005Metric, symbol UPduino_v3.0:Device_R
- removed U3: TL431DBZ, Package_TO_SOT_SMD:SOT-23, symbol Reference_Voltage:TL431DBZ
- added C48, C49, C51, C63, C73, C74: 0.1u, Capacitor_SMD:C_0201_0603Metric, symbol Device:C
- added C62: 4.7u, Capacitor_SMD:C_0402_1005Metric, symbol Device:C
- added C68: 2.2u, Capacitor_SMD:C_0402_1005Metric, symbol Device:C
- added D3: LED, symbol Device:LED
- added D5: LTST-C191KGKT, LED_SMD:LED_0603_1608Metric, symbol UPduino_v3.0:Device_LED_ALT
- added D7: MHPA1010RGBDT, CUSTOM:LED_Cree-PLCC4_1x1mm_CW, symbol UPduino_v3.0:Device_LED_ARGB
- added IC1: LP5810ADSDR, symbol SamacSys:LP5810ADSDR
- added J2: SM03B-SRSS-TB, Connector_JST:JST_SH_SM03B-SRSS-TB_1x03-1MP_P1.00mm_Horizontal, symbol Connector_Generic_MountingPin:Conn_01x03_MountingPin
- added JP3: SolderJumper_3_Bridged12, Jumper:SolderJumper-3_P1.3mm_Bridged12_RoundedPad1.0x1.5mm, symbol Jumper:SolderJumper_3_Bridged12
- added JP4, JP9: SolderJumper_2_Bridged, Jumper:SolderJumper-2_P1.3mm_Bridged_RoundedPad1.0x1.5mm, symbol Jumper:SolderJumper_2_Bridged
- added R17, R35: DNF, Resistor_SMD:R_0402_1005Metric, symbol Device:R_Small
- added R40, R42, R55, R60, R63, R70, R71: 10K, Resistor_SMD:R_0402_1005Metric, symbol Device:R_Small
- added R41, R49: 2.2K, Resistor_SMD:R_0402_1005Metric, symbol Device:R_Small
- added R43: 100, Resistor_SMD:R_0402_1005Metric, symbol Device:R_Small
- added R52: 200K, Resistor_SMD:R_0402_1005Metric, symbol Device:R
- added R56, R57, R58: 1K, Resistor_SMD:R_0402_1005Metric, symbol Device:R
- added SW1: CS1213AGF260, CUSTOM:PTS820J25KSMTRLFS, symbol Switch:SW_Push
- added U8: TXS0108EPW, Package_SO:TSSOP-20_4.4x6.5mm_P0.65mm, symbol Logic_LevelTranslator:TXS0108EPW
- added U9: APS6404L-3SQN-SN, Package_SO:SOIC-8_3.9x4.9mm_P1.27mm, symbol UPduino_v3.0:W25Q32JVSS-Memory_Flash
- C52: renamed from C1; footprint Capacitor_SMD:C_0402_1005Metric -> Capacitor_SMD:C_0201_0603Metric; symbol UPduino_v3.0:Device_C -> Device:C
- C53: renamed from C2; symbol UPduino_v3.0:Device_C -> Device:C
- C54: renamed from C3; symbol UPduino_v3.0:Device_C -> Device:C
- C55: renamed from C4; footprint Capacitor_SMD:C_0402_1005Metric -> Capacitor_SMD:C_0201_0603Metric
- C56: renamed from C5; footprint Capacitor_SMD:C_0402_1005Metric -> Capacitor_SMD:C_0201_0603Metric
- C57: renamed from C6; symbol UPduino_v3.0:Device_C -> Device:C
- C58: renamed from C7; symbol UPduino_v3.0:Device_C -> Device:C
- C59: renamed from C8; footprint Capacitor_SMD:C_0402_1005Metric -> Capacitor_SMD:C_0201_0603Metric; symbol UPduino_v3.0:Device_C -> Device:C
- C60: renamed from C9; footprint Capacitor_SMD:C_0402_1005Metric -> Capacitor_SMD:C_0201_0603Metric; symbol UPduino_v3.0:Device_C -> Device:C
- C61: renamed from C10; symbol UPduino_v3.0:Device_C -> Device:C
- C64: renamed from C11; symbol UPduino_v3.0:Device_C -> Device:C
- C65: renamed from C12; footprint Capacitor_SMD:C_0402_1005Metric -> Capacitor_SMD:C_0201_0603Metric; symbol UPduino_v3.0:Device_C -> Device:C
- C66: renamed from C14; footprint Capacitor_SMD:C_0402_1005Metric -> Capacitor_SMD:C_0201_0603Metric; symbol UPduino_v3.0:Device_C -> Device:C
- C67: renamed from C15; footprint Capacitor_SMD:C_0402_1005Metric -> Capacitor_SMD:C_0201_0603Metric; symbol UPduino_v3.0:Device_C -> Device:C
- C69: renamed from C17; footprint Capacitor_SMD:C_0402_1005Metric -> Capacitor_SMD:C_0201_0603Metric; symbol UPduino_v3.0:Device_C -> Device:C
- C70: renamed from C18; footprint Capacitor_SMD:C_0402_1005Metric -> Capacitor_SMD:C_0201_0603Metric; symbol UPduino_v3.0:Device_C -> Device:C
- C71: renamed from C19; footprint Capacitor_SMD:C_0402_1005Metric -> Capacitor_SMD:C_0201_0603Metric; symbol UPduino_v3.0:Device_C -> Device:C
- C72: renamed from C20; footprint Capacitor_SMD:C_0402_1005Metric -> Capacitor_SMD:C_0201_0603Metric; symbol UPduino_v3.0:Device_C -> Device:C
- R34: renamed from R1; value 1k -> 1K
- R45: renamed from R3; value 1k -> 1K
- R50: renamed from R8; symbol Device:R -> Device:R_Small
- R51: renamed from R9; symbol UPduino_v3.0:Device_R -> Device:R
- SJ2: renamed from SJ1; symbol UPduino_v3.0:Device_R -> Device:R
- renumbered D2 to D4, L1 to L4, R2 to R44, R5 to R46, R6 to R47, R7 to R48, R12 to R53, R13 to R54, SW1 to SW2, U1 to U10, U2 to U11, Y1 to Y2
Connections:
- net ADC5|VREF is gone; now on net ADC1: U11.56 (GPIO45_ADC5)
- net ADC6 is gone; now on net RP_BUTTONn: U11.57 (GPIO46_ADC6)
- net ~{SRAM_SS} is gone; now on net LED.B: U11.6 (GPIO8)
- net ADC1: no longer U11.52 (GPIO41_ADC1)
- net GND: now also C48.2, C49.2, C51.2, C62.2, C63.2, C68.2, C73.2, C74.2, IC1.2 (SYNC), IC1.9 (GND), J2.2 (Pin_2), J2.MP (MountPin), R52.2, SW1.2, U8.11 (GND), U9.4 (GND); no longer SW2.SH1, SW2.SH2
- net P3V3D: now also C49.1, C51.1, C62.1, C63.1, JP9.2 (B), R17.2, R35.2, R40.2, R41.2, R42.2, U8.19 (VCCB), U9.8 (VCC); no longer C64.1, C65.1, C66.1, C67.1, C69.1, C70.1, C71.1, C72.1, U11.15 (IOVDD), U11.24 (IOVDD), U11.29 (IOVDD), U11.41 (IOVDD), U11.5 (IOVDD), U11.50 (IOVDD), U11.60 (IOVDD), U11.76 (IOVDD)
- net P3V3A_VREF: now reaches U11.59 (ADC_AVDD)
- net P3V3A_VREF: now also C68.1, C74.1, JP9.1 (A)
- net SHARED_PMOD_A3: now reaches U11.22 (GPIO22)
- net SHARED_PMOD_A0: now reaches U11.21 (GPIO21)
- net LED.R: now reaches U11.3 (GPIO6)
- net LED.R: now also R46.1
- net ADC2|PB renamed RP_BUTTONn
- net RP_BUTTONn: no longer U11.53 (GPIO42_ADC2)
- net ADC3 renamed RP_MOSI_1V8
- net RP_MOSI_1V8: now also R70.2, U8.4 (A3)
- net ADC4 renamed ADC0
- net ADC7 renamed QSPI_SRAM_CSn_1V8
- net QSPI_SRAM_CSn_1V8: now also R71.2, U8.7 (A6)
- net GPIO10 renamed SHARED_PMOD_EN
- net GPIO11 renamed DONE
- net DONE: now also D5.2 (A), R49.2
- net ICE_11 renamed SHARED_PMOD_B0
- net ICE_18 renamed SHARED_PMOD_A5
- net ICE_19 renamed SHARED_PMOD_A1
- net ICE_21 renamed SHARED_PMOD_A7
- net ICE_23 renamed SHARED_PMOD_A4
- net ICE_25 renamed SHARED_PMOD_B3
- net ICE_26 renamed SHARED_PMOD_A6
- net ICE_27 renamed SHARED_PMOD_A2
- net ICE_9 renamed SHARED_PMOD_B2
- net ICE_DONE|ADC0 renamed RP_SPI.MISO
- net ICE_SI renamed I2C0.SDA
- net ICE_SO renamed LED.G
- net LED.G: now also R47.1
- net ICE_SSN renamed I2C0.SCL
- net L0_N renamed HSTX1
- net L0_P renamed HSTX0
- net L1_N renamed HSTX3
- net L1_P renamed HSTX2
- net L2_N renamed HSTX5
- net L2_P renamed HSTX4
- net L3_N renamed HSTX7
- net L3_P renamed HSTX6
- net LED_B renamed LED.B
- net LED.B: no longer U11.7 (GPIO9)
- net LED_G renamed QSPI.CSn
- net QSPI.CSn: no longer R47.1
- net LED_R renamed I2C_IRQn
- net I2C_IRQn: no longer R46.1
- net PICO_PMOD_A1 renamed SHARED_PMOD_B4
- net PICO_PMOD_A2 renamed SHARED_PMOD_B5
- net PICO_PMOD_A3 renamed SHARED_PMOD_B6
- net PICO_PMOD_A4 renamed SHARED_PMOD_B7
- net PICO_PMOD_B1 renamed FPGA_CLK_EN
- net PICO_PMOD_B2 renamed FPGA_EN
- net PICO_PMOD_B3 renamed JTAG_ENn
- net PICO_PMOD_B4 renamed MULTI_FN
- net MULTI_FN: now also D3.1 (K), R42.1, R43.2
- net QSPI_SCLK renamed QSPI.SCLK
- net QSPI.SCLK: now also U9.6 (CLK)
- net QSPI_SD0 renamed QSPI.SD0
- net QSPI.SD0: now also U9.5 (DI(IO0))
- net QSPI_SD1 renamed QSPI.SD1
- net QSPI.SD1: now also U9.2 (DO(IO1))
- net QSPI_SD2 renamed QSPI.SD2
- net QSPI.SD2: now also U9.3 (IO2)
- net QSPI_SD3 renamed QSPI.SD3
- net QSPI.SD3: now also U9.7 (IO3)
- net SCL_GPIO3 renamed I2C1.SCL
- net I2C1.SCL: now also IC1.3 (SCL)
- net SDA_GPIO2 renamed I2C1.SDA
- net I2C1.SDA: now also JP4.1 (A)
- net SWCLK renamed SWDCLK
- net SWDCLK: now also U8.5 (A4)
- net SWD renamed SWDIO
- net SWDIO: now also U8.6 (A5)
- net USB_D+ renamed USB.D+
- net USB_D- renamed USB.D-
- net USB_N: no longer names the net of R54.2, U11.66 (USB_DM)
- net USB_P: no longer names the net of R53.2, U11.67 (USB_DP)
- net VREG_AVDD: no longer names the net of C58.1, R44.1, U11.61 (VREG_AVDD)
- net VREG_LX: no longer names the net of L4.2, U11.63 (VREG_LX)
- net V_{in} renamed P5VD
- net P5VD: now also C73.1, D7.1 (A), IC1.1 (VCC)
- net ~{ICE_RST} renamed SHARED_PMOD_B1
- net ~{QSPI_SS} renamed QSPI_FLASH_CSn
- net QSPI_FLASH_CSn: now also R17.1
- net ~{RESET} renamed RESETn
- net RESETn: now also JP3.3 (B), R40.1
- net ~{USB_BOOT} renamed USB_BOOTn
- new net: JP3.2 (C), SW1.1
- new net: D3.2 (A), R41.1
- new net: JP3.1 (A), R43.1
- new net: J2.1 (Pin_1), U8.16 (B4)
- new net: J2.3 (Pin_3), U8.15 (B5)
- new net: R55.2, U8.10 (OE)
- new net: D7.4 (BK), R58.1
- new net: IC1.6 (OUT2), R58.2
- new net: D7.2 (RK), R56.1
- new net: D7.3 (GK), R57.1
- new net: IC1.7 (OUT1), R57.2
- new net: IC1.4 (SDA), JP4.2 (B)
- new net: IC1.8 (OUT0), R56.2
- new net EXT_LED: IC1.5 (OUT3)
- new net FPC_IO.LED_EN: U8.13 (B7)
- new net FPC_IO.PWR_EN: R52.1, U8.12 (B8)
- new net FPC_IO_1V8.LED_EN: U8.8 (A7)
- new net FPC_IO_1V8.PWR_EN: U8.9 (A8)
- new net LED.MONO: D5.1 (K), U11.7 (GPIO9)
- new net P1V8D: C48.1, C64.1, C65.1, C66.1, C67.1, C69.1, C70.1, C71.1, C72.1, R55.1, R60.1, R63.1, R70.1, R71.1, U11.15 (IOVDD), U11.24 (IOVDD), U11.29 (IOVDD), U11.41 (IOVDD), U11.5 (IOVDD), U11.50 (IOVDD), U11.60 (IOVDD), U11.76 (IOVDD), U8.2 (VCCA)
- new net P3V3D_FPGA: R49.1
- new net QSPI_SRAM_CSn: R35.1, U8.14 (B6), U9.1 (~{CS})
- new net RP_CSn_1V8: R60.2, U11.52 (GPIO41_ADC1), U8.1 (A1)
- new net RP_SCK_1V8: R63.2, U11.53 (GPIO42_ADC2), U8.3 (A2)
- new net RP_SPI.CSn: U8.20 (B1)
- new net RP_SPI.MOSI: U8.17 (B3)
- new net RP_SPI.SCK: U8.18 (B2)
- no-connect marks 2 -> 0
Other:
- note added: "Although the level shifter has internal pull-ups, they are relatively weak at 40K. During RP boot, its internal pull-downs are 50-80K, which would lead to an indeterminate logic level, if it weren't for the strong 10K external pull-ups."
- note added: "Button"
- note added: "Crystal oscillator instead of MEMS oscillator so it can be disabled without additional IO."
- note added: "Flash"
- note added: "I2C Constant Current LED Driver"
- note added: "Level Shifter"
- note added: "Mono LED"
- note added: "Multi-Function IO"
- note added: "P3V3A_VREF can be connected to an external voltage reference."
- note added: "RGB LED"
- note added: "RP2350"
- note added: "Reset state of SWDIO and SWDCLK is pull-up"
- note added: "SRAM"
- note added: "This LED can be used for any purpose but it can not illuminate unless the FPGA is in user mode."
- note added: "USB series termination close to RP2040"
- note removed: "FPGA Clock"
- note removed: "Hold FPGA in reset while the pico is coming up"
- note removed: "I_{KA} (Cathode current) > 0.5mA"
- note removed: "Note: Set the GPIO high to enable power to the reference when the ADC needs to be calibrated. Remove resistors to use the ADC on the external pins."
- note removed: "PICO Button"
- note removed: "Peripheral(Default)/Host Selection Host Mode: Solder open bridges, cut shorted bridges Peripheral: Default"
- note removed: "Pico Flash"
- note removed: "Place R4/R5 close to RP2040"
- note removed: "Power monitor"
- note removed: "RP2 LED"
- note removed: "Raspberry Pico"
- note removed: "Suggested data clock"
- note removed: "USBC Connector"
- note removed: "V_{ref} = 2.5V"
- moved on the sheet: C52, C53, C54, C55, C56, C57, C58, C59, C60, C61, C64, C65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
