File: board/Rev0/pico2-nx/pico2-nx.kicad_sch (KiCad schematic)
At the start: 0 parts

Commit message: draft rev 0 work in progress
Parts:
- added R1, R2, R3, R4: 10K, Resistor_SMD:R_0402_1005Metric, symbol Device:R_Small
- added R14: 200K, Resistor_SMD:R_0402_1005Metric, symbol Device:R_Small
- added R5, R6, R7, R8: 4.7K, Resistor_SMD:R_0402_1005Metric, symbol Device:R_Small
Connections:
- new net Connectors/FPGA_EN: R14.2
- new net Connectors/I2C_IRQn: R4.1
- new net EXT_SPI.CSn: R3.1
- new net EXT_SPI.MOSI: R1.1
- new net EXT_SPI.SCK: R2.1
- new net GND: R14.1
- new net I2C0.SCL: R8.1
- new net I2C0.SDA: R7.1
- new net I2C1.SCL: R6.1
- new net I2C1.SDA: R5.1
- new net P3V3D: R4.2, R5.2, R6.2, R7.2, R8.2
- new net P3V3D_FPGA: R1.2, R2.2, R3.2
Other:
- sheet Connectors ports: added ADC[0..1], DONE, EXT_LED, EXT_MIPI{D0+ D0- D1+ D1- D2+ D2- D3+ D3- CLK+ CLK-}, EXT_SPI{CSn SCK MOSI MISO}, FPC_IO{PWR_EN LED_EN}, FPGA_CLK_EN, FPGA_EN, FPGA_PMOD[0..7], I2C0{SCL SDA}, I2C1{SCL SDA}, I2C_IRQn, LED{R G B MONO}, MULTI_FN, PWR_EN, RESETn, RGB_MIPI{D0+ D0- D1+ D1- D2+ D2- D3+ D3- CLK+ CLK-}, RP_SPI{CSn SCK MOSI MISO}, SHARED_PMOD_A[0..7], SHARED_PMOD_B[0..7], SHARED_PMOD_EN, UJTAG{PRESENTn TCK TMS TDI TDO}, USB_BOOTn, USB{D+ D-}; removed none
- sheet FPGA ports: added DONE, EXT_MIPI{D0+ D0- D1+ D1- D2+ D2- D3+ D3- CLK+ CLK-}, EXT_SPI{CSn SCK MOSI MISO}, FPC_IO_1V8{PWR_EN LED_EN}, FPGA_CLK_EN, FPGA_PMOD[0..7], HSTX[0..7], I2C1{SCL SDA}, I2C_IRQn, JTAG_ENn, MULTI_FN, QSPI{CSn SCLK SD0 SD1 SD2 SD3}, RGB_MIPI{D0+ D0- D1+ D1- D2+ D2- D3+ D3- CLK+ CLK-}, SHARED_PMOD_A[0..7], SHARED_PMOD_B[0..7], UJTAG{PRESENTn TCK TMS TDI TDO}; removed FPGA_RESETn, HSTX
- sheet RP2350 ports: added ADC[0..1], DONE, EXT_LED, FPC_IO_1V8{PWR_EN LED_EN}, FPC_IO{PWR_EN LED_EN}, FPGA_CLK_EN, FPGA_EN, HSTX[0..7], I2C0{SCL SDA}, I2C1{SCL SDA}, I2C_IRQn, JTAG_ENn, LED{R G B MONO}, MULTI_FN, QSPI{CSn SCLK SD0 SD1 SD2 SD3}, RESETn, RP_SPI{CSn SCK MOSI MISO}, SHARED_PMOD_A[0..7], SHARED_PMOD_B[0..7], SHARED_PMOD_EN, USB_BOOTn, USB{D+ D-}; removed HSTX
- note added: "P5VD"
- note added: "TODO: - additional ESD protection? - should 3.3V be a switcher or an LDO?"
- note removed: "V_{in}"
- company: (none) -> tinyVision.ai Inc.
- title: (none) -> PICO2-NX
